File: driver2110.kicad_pcb (KiCad board)
At the start: 2 copper layers, 40 parts, among them J1 Screw_Terminal_01x03, J10 Conn_01x03_Male, J2 Conn_01x07_Male, J6 Conn_01x03_Male, J9 Conn_01x03_Male, U1 74HC14, U3 IR2110, U6 IR2110, U9 IR2110

Commit message: Correccion en la comprobacion del esquematico
para corregir los errores, se agregaron librerías, modificaron los cableados y se pusieron test points
Parts:
- removed J10, J6, J9: Conn_01x03_Male, Connector:FanPinHeader_1x03_P2.54mm_Vertical
- removed the REF** at (91.9, 132.1)
- removed the REF** at (46.2, 39.5)
- removed the REF** at (184.4, 39.4)
- added A1: ESP32_DevKit_V1_DOIT_30GPIOs, ESP32-DEVKITC:MODULE_ESP32-DEVKITC, F.Cu at (-248.9, 91.4)
- added C10: 10uf, Capacitor_THT:C_Axial_L5.1mm_D3.1mm_P7.50mm_Horizontal, F.Cu at (-45.8, 39.7)
- added C11: 0.1uf, Capacitor_THT:C_Axial_L5.1mm_D3.1mm_P7.50mm_Horizontal, F.Cu at (-45.8, 44.4)
- added D10: 1N4148, 1N4007-Diotec-Symbol-Kicad-711646:P1_DO-41, F.Cu at (-157.5, 47.1)
- added D11: 1N4007, 1N4007-Diotec-Symbol-Kicad-711646:P1_DO-41, F.Cu at (-157.5, 51.0)
- added D12: 1N4148, 1N4007-Diotec-Symbol-Kicad-711646:P1_DO-41, F.Cu at (-157.5, 54.9)
- added D13: 1N4007, 1N4007-Diotec-Symbol-Kicad-711646:P1_DO-41, F.Cu at (-157.5, 58.8)
- added D14: 1N4148, 1N4007-Diotec-Symbol-Kicad-711646:P1_DO-41, F.Cu at (-157.5, 62.7)
- added D15: 1N4007, 1N4007-Diotec-Symbol-Kicad-711646:P1_DO-41, F.Cu at (-157.5, 66.6)
- added D4: 1N4148, 1N4007-Diotec-Symbol-Kicad-711646:P1_DO-41, F.Cu at (-157.5, 23.6)
- added D5: 1N4007, 1N4007-Diotec-Symbol-Kicad-711646:P1_DO-41, F.Cu at (-157.5, 27.5)
- added D6: 1N4148, 1N4007-Diotec-Symbol-Kicad-711646:P1_DO-41, F.Cu at (-157.5, 31.4)
- added D7: 1N4007, 1N4007-Diotec-Symbol-Kicad-711646:P1_DO-41, F.Cu at (-157.5, 35.4)
- added D8: 1N4148, 1N4007-Diotec-Symbol-Kicad-711646:P1_DO-41, F.Cu at (-157.5, 39.3)
- added D9: 1N4007, 1N4007-Diotec-Symbol-Kicad-711646:P1_DO-41, F.Cu at (-157.5, 43.2)
- added J1: Screw_Terminal_01x03, TerminalBlock:TerminalBlock_bornier-3_P5.08mm, F.Cu at (-44.1, 32.9)
- added Q1: IRF840, IRF840:TO220, F.Cu at (-130.9, 173.7)
- added Q2: IRF840, IRF840:TO220, F.Cu at (-119.4, 173.7)
- added Q3: IRF840, IRF840:TO220, F.Cu at (-107.8, 173.7)
- added Q4: IRF840, IRF840:TO220, F.Cu at (-83.6, 178.3)
- added Q5: IRF840, IRF840:TO220, F.Cu at (-72.1, 178.3)
- added Q6: IRF840, IRF840:TO220, F.Cu at (-78.7, 217.2)
- added R1: Resistor, Resistor_THT:R_Axial_DIN0207_L6.3mm_D2.5mm_P10.16mm_Horizontal, F.Cu at (-59.1, 30.4)
- added R2: Resistor, Resistor_THT:R_Axial_DIN0207_L6.3mm_D2.5mm_P10.16mm_Horizontal, F.Cu at (-59.1, 34.4)
- added R3: Resistor, Resistor_THT:R_Axial_DIN0207_L6.3mm_D2.5mm_P10.16mm_Horizontal, F.Cu at (-59.1, 38.5)
- added R4: Resistor, Resistor_THT:R_Axial_DIN0207_L6.3mm_D2.5mm_P10.16mm_Horizontal, F.Cu at (-59.1, 42.5)
- added R5: Resistor, Resistor_THT:R_Axial_DIN0207_L6.3mm_D2.5mm_P10.16mm_Horizontal, F.Cu at (-59.1, 46.6)
- added R6: Resistor, Resistor_THT:R_Axial_DIN0207_L6.3mm_D2.5mm_P10.16mm_Horizontal, F.Cu at (-59.1, 50.6)
- added REF**: MountingHole_3.2mm_M3, MountingHole:MountingHole_3.2mm_M3, F.Cu at (93.5, 40.6)
- added REF**: MountingHole_3.2mm_M3, MountingHole:MountingHole_3.2mm_M3, F.Cu at (233.7, 40.6)
- added REF**: MountingHole_3.2mm_M3, MountingHole:MountingHole_3.2mm_M3, F.Cu at (93.5, 130.8)
- D1, D2, D3: footprint Diode_THT:D_DO-41_SOD81_P10.16mm_Horizontal -> 1N4007-Diotec-Symbol-Kicad-711646:P1_DO-41
- moved C7 164.3 mm to (-38.1, 178.1)
- moved D4 164.3 mm to (-45.7, 167.6)
- moved R1 164.3 mm to (-45.7, 172.7)
- moved C1 65.0 mm to (217.4, 64.8)
- moved C3 65.0 mm to (216.6, 92.0)
- moved C5 65.0 mm to (216.1, 116.9)
- moved C8 65.0 mm to (181.0, 63.8)
- moved D1 65.0 mm to (224.0, 109.5)
- moved D3 65.0 mm to (225.2, 57.2)
- moved J2 65.0 mm to (163.3, 81.3)
- moved R4 65.0 mm to (193.0, 102.4)
- moved TP4 65.0 mm to (193.0, 94.5)
- moved TP6 65.0 mm to (193.0, 86.7)
- moved C9 65.0 mm to (180.5, 46.3)
- moved D5 65.0 mm to (173.2, 58.2)
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Connections:
- C2 pad 2: VDD -> Net-(D3-A)
- C4 pad 2: VDD -> Net-(D2-A)
- C6 pad 2: VDD -> Net-(D1-A)
- C7 pad 1: Net-(C7-Pad1) -> VCC
- C8 pad 1: Net-(C8-Pad1) -> VCC
- C9 pad 1: Net-(C9-Pad1) -> VCC
- D1 pad 2: VDD -> Net-(D1-A)
- D2 pad 2: VDD -> Net-(D2-A)
- D3 pad 2: VDD -> Net-(D3-A)
- TP1 pad 1: Net-(TP1-Pad1) -> /INLC
- TP2 pad 1: Net-(C7-Pad1) -> /INHC
- TP3 pad 1: Net-(TP3-Pad1) -> /INLA
- TP4 pad 1: Net-(TP4-Pad1) -> /INLB
- TP5 pad 1: Net-(C9-Pad1) -> /INHA
- TP6 pad 1: Net-(C8-Pad1) -> /INHB
- U3 pad 10: Net-(C9-Pad1) -> /INHA
- U3 pad 12: Net-(TP3-Pad1) -> /INLA
- U3 pad 3: VDD -> Net-(D3-A)
- U6 pad 10: Net-(C8-Pad1) -> /INHB
- U6 pad 12: Net-(TP4-Pad1) -> /INLB
- U6 pad 3: VDD -> Net-(D2-A)
- U9 pad 10: Net-(C7-Pad1) -> /INHC
- U9 pad 12: Net-(TP1-Pad1) -> /INLC
- U9 pad 3: VDD -> Net-(D1-A)
Routing:
- net VSS: track 305.7 -> 254.6 mm
- net Net-(D10-K): track 45.4 -> 3.68 mm
- net Net-(D6-K): track 44.2 -> 4.25 mm
- net Net-(D12-K): track 41.0 -> 2.51 mm
- net Net-(D14-K): track 41.6 -> 4.10 mm
- net Net-(D8-K): track 43.0 -> 5.54 mm
- net Net-(D4-K): track 41.8 -> 4.82 mm
- net Net-(J1-Pin_3): track 36.5 -> 0.00 mm
- net Net-(C7-Pad1): track 33.7 -> 0.00 mm
- net /INHC: track 0.00 -> 33.7 mm
- net Net-(U3-VS): track 36.1 -> 7.91 mm
- net Net-(Q3-S): track 37.3 -> 13.0 mm
- net Net-(D4-Pad1): track 38.8 -> 19.4 mm
- net (no net): track 0.00 -> 16.3 mm
- net VDD: track 172.4 -> 161.0 mm
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- removed copper zone on B.Cu, net GND
- removed copper zone on B.Cu, net VSS
